File: hardware/electronics/drvPcb/drvPcb.kicad_pcb (KiCad board)
At the start: 2 copper layers, 100 x 54.6 mm, 13 parts, among them J1 Conn_01x03_Male, J2 Conn_01x03_Male, J3 Conn_01x02_Female, J4 Conn_01x02_Female, J5 Conn_01x03_Female, J6 silent step stick, J7 silent step stick, Q1 AO3400A, Q2 AO3400A, Q3 AO3400A, Q4 AO3400A, U1 Pico

Commit message: ...
Parts:
- removed REF**: Jack_3.5mm_Lumberg_1503_02_Horizontal, Connector_Audio:Jack_3.5mm_Lumberg_1503_02_Horizontal
- added C45: 100nF, Capacitor_SMD:C_1206_3216Metric_Pad1.33x1.80mm_HandSolder, B.Cu at (135.6, 80.3)
- added C46: 100nF, Capacitor_SMD:C_1206_3216Metric_Pad1.33x1.80mm_HandSolder, B.Cu at (159.8, 61.1)
- added D1: 1N4148WS, Diode_SMD:D_1206_3216Metric_Pad1.42x1.75mm_HandSolder, B.Cu at (154.2, 80.1)
- added D2: D, Diode_SMD:D_1206_3216Metric_Pad1.42x1.75mm_HandSolder, B.Cu at (132.4, 93.5)
- added D3: D, Diode_SMD:D_1206_3216Metric_Pad1.42x1.75mm_HandSolder, B.Cu at (145.6, 93.8)
- added D4: D, Diode_SMD:D_1206_3216Metric_Pad1.42x1.75mm_HandSolder, B.Cu at (132.2, 110.6)
- added D5: D, Diode_SMD:D_1206_3216Metric_Pad1.42x1.75mm_HandSolder, B.Cu at (145.5, 110.6)
- added D6: D, Diode_SMD:D_1206_3216Metric_Pad1.42x1.75mm_HandSolder, B.Cu at (83.9, 121.6)
- added DCDC1: ~, Library:Converter_DCDC, F.Cu at (163.5, 77.8)
- added IC8: H11L1, Package_DIP:SMDIP-6_W9.53mm, F.Cu at (146.8, 79.0)
- added J10: Servo1, Library:PinHeader_1x03_P2.54mm_Vertical(fmod), F.Cu at (51.4, 123.2)
- added J11: Servo1, Library:PinHeader_1x03_P2.54mm_Vertical(fmod), F.Cu at (71.7, 123.2)
- added J12: Conn_01x03_Socket, Library:PinHeader_1x03_P2.54mm_Vertical(fmod), F.Cu at (67.3, 83.3)
- added J13: Analog_2, Library:PinHeader_1x03_P2.54mm_Vertical(fmod), F.Cu at (114.4, 72.9)
- added J14: endstp2, Library:PinHeader_1x02_P2.54mm_Vertical_(fmod), F.Cu at (61.8, 108.6)
- added J15: Servo1, Library:PinHeader_1x03_P2.54mm_Vertical(fmod), F.Cu at (67.6, 123.2)
- added J16: Servo1, Library:PinHeader_1x03_P2.54mm_Vertical(fmod), F.Cu at (63.6, 123.2)
- added J17: Servo1, Library:PinHeader_1x03_P2.54mm_Vertical(fmod), F.Cu at (55.4, 123.2)
- added J18: Servo1, Library:PinHeader_1x03_P2.54mm_Vertical(fmod), F.Cu at (59.5, 123.2)
- added J19: Analog_1, Library:PinHeader_1x03_P2.54mm_Vertical(fmod), F.Cu at (114.4, 76.7)
- added J20: 5v jack, Library:PinHeader_1x02_P2.54mm_Vertical_(fmod), F.Cu at (119.4, 61.5)
- added J21: AudioJack3, Library:Jack_3.5mm_CUI_SJ1-3523N_Horizontal(fmod), F.Cu at (150.9, 60.7)
- added J22: Conn_01x03_Socket, Library:PinHeader_1x03_P2.54mm_Vertical(fmod), F.Cu at (62.8, 75.7)
- added J23: Conn_01x03_Socket, Library:PinHeader_1x03_P2.54mm_Vertical(fmod), F.Cu at (62.8, 79.5)
- added J24: Conn_01x03_Socket, Library:PinHeader_1x03_P2.54mm_Vertical(fmod), F.Cu at (67.3, 79.5)
- added J25: Conn_01x03_Socket, Library:PinHeader_1x03_P2.54mm_Vertical(fmod), F.Cu at (62.8, 83.3)
- added J28: Conn_01x03_Socket, Library:PinHeader_1x03_P2.54mm_Vertical(fmod), F.Cu at (67.3, 75.5)
- added J29: silent step stick, Library:stepstick, F.Cu at (74.0, 94.2)
- added J31: stp2_conn., Library:PinHeader_1x04_P2.54mm_Vertical(fmod), F.Cu at (51.4, 97.3)
- added J9: AudioJack3, Library:Jack_3.5mm_CUI_SJ1-3523N_Horizontal(fmod), F.Cu at (137.1, 60.7)
- added J_mf1: socket 2, Library:PinHeader_1x02_P2.54mm_Vertical_(fmod), F.Cu at (136.2, 95.0)
- added J_mf2: socket 2, Library:PinHeader_1x02_P2.54mm_Vertical_(fmod), F.Cu at (141.8, 92.5)
- added J_mf3: socket 2, Library:PinHeader_1x02_P2.54mm_Vertical_(fmod), F.Cu at (136.2, 111.9)
- added J_mf4: socket 2, Library:PinHeader_1x02_P2.54mm_Vertical_(fmod), F.Cu at (141.7, 109.3)
- added Q5: AO3400A, Package_TO_SOT_SMD:SOT-223-3_TabPin2, B.Cu at (90.8, 121.3)
- added R1: 10k, Resistor_SMD:R_1206_3216Metric_Pad1.30x1.75mm_HandSolder, B.Cu at (119.4, 92.8)
- added R10: 10k, Resistor_SMD:R_1206_3216Metric_Pad1.30x1.75mm_HandSolder, B.Cu at (158.7, 111.2)
- added R11: 200, Resistor_SMD:R_1206_3216Metric_Pad1.30x1.75mm_HandSolder, B.Cu at (95.6, 116.0)
- added R12: 10k, Resistor_SMD:R_1206_3216Metric_Pad1.30x1.75mm_HandSolder, B.Cu at (97.3, 120.5)
- added R2: 200, Resistor_SMD:R_1206_3216Metric_Pad1.30x1.75mm_HandSolder, B.Cu at (116.9, 92.7)
- added R20: 33, Resistor_SMD:R_1206_3216Metric_Pad1.30x1.75mm_HandSolder, B.Cu at (132.6, 80.3)
- added R21: 270, Resistor_SMD:R_1206_3216Metric_Pad1.30x1.75mm_HandSolder, B.Cu at (138.6, 80.3)
- added R22: 220, Resistor_SMD:R_1206_3216Metric_Pad1.30x1.75mm_HandSolder, B.Cu at (157.2, 80.0)
- added R23: 10, Resistor_SMD:R_1206_3216Metric_Pad1.30x1.75mm_HandSolder, B.Cu at (128.0, 64.1)
- added R3: 200, Resistor_SMD:R_1206_3216Metric_Pad1.30x1.75mm_HandSolder, B.Cu at (150.8, 100.6)
- added R4: 10k, Resistor_SMD:R_1206_3216Metric_Pad1.30x1.75mm_HandSolder, B.Cu at (158.8, 94.5)
- added R5: 10k, Resistor_SMD:R_1206_3216Metric_Pad1.30x1.75mm_HandSolder, B.Cu at (54.9, 107.6)
- added R6: 10k, Resistor_SMD:R_1206_3216Metric_Pad1.30x1.75mm_HandSolder, B.Cu at (58.0, 107.6)
- added R7: 200, Resistor_SMD:R_1206_3216Metric_Pad1.30x1.75mm_HandSolder, B.Cu at (116.8, 110.0)
- added R8: 10k, Resistor_SMD:R_1206_3216Metric_Pad1.30x1.75mm_HandSolder, B.Cu at (119.4, 109.9)
- added R9: 200, Resistor_SMD:R_1206_3216Metric_Pad1.30x1.75mm_HandSolder, B.Cu at (150.7, 117.3)
- J1: value Conn_01x03_Male -> Barrel_Jack_in; footprint Connector_PinHeader_2.54mm:PinHeader_1x03_P2.54mm_Vertical -> Library:BarrelJack_GCT_DCJ200-10-A_Horizontal(fmod)
- J2: value Conn_01x03_Male -> Barrel_Jack_out; footprint Connector_PinHeader_2.54mm:PinHeader_1x03_P2.54mm_Vertical -> Library:BarrelJack_GCT_DCJ200-10-A_Horizontal(fmod)
- J3, J4: value Conn_01x02_Female -> Servo1; footprint Connector_PinHeader_2.54mm:PinHeader_1x02_P2.54mm_Vertical -> Library:PinHeader_1x03_P2.54mm_Vertical(fmod)
- J5: value Conn_01x03_Female -> endstp1; footprint Connector_PinHeader_2.54mm:PinHeader_1x03_P2.54mm_Vertical -> Library:PinHeader_1x02_P2.54mm_Vertical_(fmod)
- J6: footprint stepstick:stepstick -> Library:stepstick
- J7: value silent step stick -> stp1_conn.; footprint stepstick:stepstick -> Library:PinHeader_1x04_P2.54mm_Vertical(fmod)
- Q1, Q2, Q3, Q4: footprint Package_TO_SOT_SMD:SOT-23 -> Package_TO_SOT_SMD:SOT-223-3_TabPin2; moved to B.Cu
- moved J4 153.2 mm to (75.8, 123.2), turned to 180 degrees
- moved J5 149.4 mm to (51.6, 108.6), turned to 180 degrees
- moved J3 145.7 mm to (79.8, 123.2), turned to 180 degrees
- moved Q3 90.3 mm to (125.8, 109.1)
- moved Q4 90.2 mm to (152.1, 112.0), turned to 180 degrees
- moved Q1 69.7 mm to (125.9, 92.1)
- moved Q2 57.5 mm to (152.2, 95.2), turned to 180 degrees
- moved U1 39.2 mm to (96.8, 83.1), turned to 0 degrees
- moved J7 30.4 mm to (51.4, 68.2), turned to 180 degrees
- moved J6 28.0 mm to (56.2, 64.5)
- moved J1 26.7 mm to (179.7, 69.7), turned to 180 degrees
- moved J2 20.6 mm to (167.4, 69.7), turned to 180 degrees
Connections:
- J1 pad 1: unconnected-(J1-Pad1) -> +24V
- J1 pad 2: unconnected-(J1-Pad2) -> GND
- J1 pad 3: unconnected-(J1-Pad3) -> (no net)
- J2 pad 1: unconnected-(J2-Pad1) -> +24V
- J2 pad 2: unconnected-(J2-Pad2) -> GND
- J2 pad 3: unconnected-(J2-Pad3) -> (no net)
- J3 pad 1: unconnected-(J3-Pad1) -> /-Servo
- J3 pad 2: unconnected-(J3-Pad2) -> +5V
- J4 pad 1: unconnected-(J4-Pad1) -> /-Servo
- J4 pad 2: unconnected-(J4-Pad2) -> +5V
- J5 pad 1: unconnected-(J5-Pad1) -> GND
- J5 pad 2: unconnected-(J5-Pad2) -> /endstp1
- J6 pad 1: unconnected-(J6-Pad1) -> /stp1_en
- J6 pad 10: unconnected-(J6-Pad10) -> +3.3V
- J6 pad 11: unconnected-(J6-Pad11) -> Net-(J6-m1b)
- J6 pad 12: unconnected-(J6-Pad12) -> Net-(J6-m1a)
- J6 pad 13: unconnected-(J6-Pad13) -> Net-(J6-m2a)
- J6 pad 14: unconnected-(J6-Pad14) -> Net-(J6-m2b)
- J6 pad 15: unconnected-(J6-Pad15) -> GND
- J6 pad 16: unconnected-(J6-Pad16) -> +24V
- J6 pad 2: unconnected-(J6-Pad2) -> Net-(J22-Pin_3)
- J6 pad 3: unconnected-(J6-Pad3) -> Net-(J22-Pin_2)
- J6 pad 4: unconnected-(J6-Pad4) -> Net-(J22-Pin_1)
- J6 pad 7: unconnected-(J6-Pad7) -> /stp1_stp
- J6 pad 8: unconnected-(J6-Pad8) -> /stp1_dir
- J7 pad 1: unconnected-(J7-Pad1) -> Net-(J6-m2b)
- J7 pad 2: unconnected-(J7-Pad2) -> Net-(J6-m2a)
- J7 pad 3: unconnected-(J7-Pad3) -> Net-(J6-m1a)
- J7 pad 4: unconnected-(J7-Pad4) -> Net-(J6-m1b)
- Q1 pad 1: unconnected-(Q1-Pad1) -> Net-(Q1-G)
- Q1 pad 2: unconnected-(Q1-Pad2) -> Net-(D2-A)
- Q1 pad 3: unconnected-(Q1-Pad3) -> GND
- Q2 pad 1: unconnected-(Q2-Pad1) -> Net-(Q2-G)
- Q2 pad 2: unconnected-(Q2-Pad2) -> Net-(D3-A)
- Q2 pad 3: unconnected-(Q2-Pad3) -> GND
- Q3 pad 1: unconnected-(Q3-Pad1) -> Net-(Q3-G)
- Q3 pad 2: unconnected-(Q3-Pad2) -> Net-(D4-A)
- Q3 pad 3: unconnected-(Q3-Pad3) -> GND
- Q4 pad 1: unconnected-(Q4-Pad1) -> Net-(Q4-G)
- Q4 pad 2: unconnected-(Q4-Pad2) -> Net-(D5-A)
- Q4 pad 3: unconnected-(Q4-Pad3) -> GND
- U1 pad 1: unconnected-(U1-Pad1) -> /stp1_en
- U1 pad 10: unconnected-(U1-Pad10) -> /endstp2
- U1 pad 11: unconnected-(U1-Pad11) -> /srv1
- U1 pad 12: unconnected-(U1-Pad12) -> /srv2
- U1 pad 14: unconnected-(U1-Pad14) -> /srv3
- U1 pad 15: unconnected-(U1-Pad15) -> /srv4
- U1 pad 16: unconnected-(U1-Pad16) -> /srv5
- U1 pad 17: unconnected-(U1-Pad17) -> /srv6
- U1 pad 18: unconnected-(U1-Pad18) -> GND
- U1 pad 19: unconnected-(U1-Pad19) -> /srv7
- U1 pad 2: unconnected-(U1-Pad2) -> /stp1_stp
- U1 pad 20: unconnected-(U1-Pad20) -> /srv8
- U1 pad 21: unconnected-(U1-Pad21) -> /MIDI_OUT
- U1 pad 22: unconnected-(U1-Pad22) -> /MIDI_IN
- U1 pad 23: unconnected-(U1-Pad23) -> GND
- U1 pad 24: unconnected-(U1-Pad24) -> /mos5_gate
- U1 pad 25: unconnected-(U1-Pad25) -> /mos4_gate
- U1 pad 26: unconnected-(U1-Pad26) -> /mos3_gate
- U1 pad 27: unconnected-(U1-Pad27) -> /mos2_gate
- U1 pad 28: unconnected-(U1-Pad28) -> GND
- U1 pad 29: unconnected-(U1-Pad29) -> /mos1_gate
- U1 pad 3: unconnected-(U1-Pad3) -> GND
- U1 pad 31: unconnected-(U1-Pad31) -> /ana2
- U1 pad 32: unconnected-(U1-Pad32) -> /ana1
- U1 pad 33: unconnected-(U1-Pad33) -> GNDA
- U1 pad 35: unconnected-(U1-Pad35) -> /ana_Vref
- U1 pad 36: unconnected-(U1-Pad36) -> +3.3V
- U1 pad 38: unconnected-(U1-Pad38) -> GND
- U1 pad 39: unconnected-(U1-Pad39) -> +5V
- U1 pad 4: unconnected-(U1-Pad4) -> /stp1_dir
- U1 pad 5: unconnected-(U1-Pad5) -> /stp2_en
- U1 pad 6: unconnected-(U1-Pad6) -> /stp2_stp
- U1 pad 7: unconnected-(U1-Pad7) -> /stp2_dir
- U1 pad 9: unconnected-(U1-Pad9) -> /endstp1
Routing:
- net +5V: track 0.00 -> 278.6 mm, vias 0 -> 5
- net /MIDI_IN: track 0.00 -> 124.0 mm
- net +24V: track 0.00 -> 105.7 mm, vias 0 -> 5
- net /MIDI_OUT: track 0.00 -> 84.0 mm
- net +3.3V: track 0.00 -> 75.2 mm, vias 0 -> 3
- net /mos4_gate: track 0.00 -> 60.7 mm
- net /srv1: track 0.00 -> 60.2 mm
- net /endstp1: track 0.00 -> 58.5 mm
- net /srv2: track 0.00 -> 49.6 mm
- net /stp2_dir: track 0.00 -> 47.7 mm
- net /mos2_gate: track 0.00 -> 47.2 mm
- net /srv3: track 0.00 -> 47.1 mm
- net /srv5: track 0.00 -> 46.8 mm
- net /srv4: track 0.00 -> 46.6 mm
- net /endstp2: track 0.00 -> 45.7 mm
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- added copper zone on B.Cu, net GND
Other:
- board size 100 x 54.6 mm -> 150 x 77 mm
