File: hardware/electronics/drvPcb/drvPcb.kicad_sch (KiCad schematic)
At the start: 12 parts, among them J1 Conn_01x03_Male, J2 Conn_01x03_Male, J3 Conn_01x02_Female, J4 Conn_01x02_Female, J5 Conn_01x03_Female, J6 silent step stick, J7 silent step stick, Q1 AO3400A, Q2 AO3400A, Q3 AO3400A, Q4 AO3400A, U1 Pico

Commit message: ...
Parts:
- removed J1, J2: Conn_01x03_Male, Connector_PinHeader_2.54mm:PinHeader_1x03_P2.54mm_Vertical, symbol Connector:Conn_01x03_Male
- removed J3, J4: Conn_01x02_Female, Connector_PinHeader_2.54mm:PinHeader_1x02_P2.54mm_Vertical, symbol Connector:Conn_01x02_Female
- removed J5: Conn_01x03_Female, Connector_PinHeader_2.54mm:PinHeader_1x03_P2.54mm_Vertical, symbol Connector:Conn_01x03_Female
- removed J7: silent step stick, stepstick:stepstick, symbol Connector_Generic:Conn_02x08_Counter_Clockwise
- added C45, C46: 100nF, Capacitor_SMD:C_1206_3216Metric_Pad1.33x1.80mm_HandSolder, symbol Device:C
- added D1: 1N4148WS, Diode_SMD:D_1206_3216Metric_Pad1.42x1.75mm_HandSolder, symbol Diode:1N4148WS
- added D2, D3, D4, D5, D6: D, Diode_SMD:D_1206_3216Metric_Pad1.42x1.75mm_HandSolder, symbol Device:D
- added DCDC1: ~, Library:Converter_DCDC, symbol drvPcb:DCDC
- added IC8: H11L1, Package_DIP:SMDIP-6_W9.53mm, symbol Isolator:H11L1
- added J1: Barrel_Jack_in, Library:BarrelJack_GCT_DCJ200-10-A_Horizontal(fmod), symbol Connector:Barrel_Jack
- added J10, J11, J15, J16, J17, J18, J3, J4: Servo1, Library:PinHeader_1x03_P2.54mm_Vertical(fmod), symbol Connector:Conn_01x03_Socket
- added J12, J22, J23, J24, J25, J28: Conn_01x03_Socket, Library:PinHeader_1x03_P2.54mm_Vertical(fmod), symbol Connector:Conn_01x03_Socket
- added J13: Analog_2, Library:PinHeader_1x03_P2.54mm_Vertical(fmod), symbol Connector:Conn_01x03_Socket
- added J14: endstp2, Library:PinHeader_1x02_P2.54mm_Vertical_(fmod), symbol Connector:Conn_01x02_Socket
- added J19: Analog_1, Library:PinHeader_1x03_P2.54mm_Vertical(fmod), symbol Connector:Conn_01x03_Socket
- added J2: Barrel_Jack_out, Library:BarrelJack_GCT_DCJ200-10-A_Horizontal(fmod), symbol Connector:Barrel_Jack
- added J20: 5v jack, Library:PinHeader_1x02_P2.54mm_Vertical_(fmod), symbol Connector:Conn_01x02_Socket
- added J21, J9: AudioJack3, Library:Jack_3.5mm_CUI_SJ1-3523N_Horizontal(fmod), symbol Connector_Audio:AudioJack3
- added J29: silent step stick, Library:stepstick, symbol Connector_Generic:Conn_02x08_Counter_Clockwise
- added J31: stp2_conn., Library:PinHeader_1x04_P2.54mm_Vertical(fmod), symbol Connector:Conn_01x04_Socket
- added J5: endstp1, Library:PinHeader_1x02_P2.54mm_Vertical_(fmod), symbol Connector:Conn_01x02_Socket
- added J7: stp1_conn., Library:PinHeader_1x04_P2.54mm_Vertical(fmod), symbol Connector:Conn_01x04_Socket
- added J_mf1, J_mf2, J_mf3, J_mf4: socket 2, Library:PinHeader_1x02_P2.54mm_Vertical_(fmod), symbol Connector:Conn_01x02_Socket
- added Q5: AO3400A, Package_TO_SOT_SMD:SOT-223-3_TabPin2, symbol Transistor_FET:AO3400A
- added R1, R10, R12, R4, R5, R6, R8: 10k, Resistor_SMD:R_1206_3216Metric_Pad1.30x1.75mm_HandSolder, symbol Device:R
- added R11, R2, R3, R7, R9: 200, Resistor_SMD:R_1206_3216Metric_Pad1.30x1.75mm_HandSolder, symbol Device:R
- added R20: 33, Resistor_SMD:R_1206_3216Metric_Pad1.30x1.75mm_HandSolder, symbol Device:R
- added R21: 270, Resistor_SMD:R_1206_3216Metric_Pad1.30x1.75mm_HandSolder, symbol Device:R
- added R22: 220, Resistor_SMD:R_1206_3216Metric_Pad1.30x1.75mm_HandSolder, symbol Device:R
- added R23: 10, Resistor_SMD:R_1206_3216Metric_Pad1.30x1.75mm_HandSolder, symbol Device:R
- J6: footprint stepstick:stepstick -> Library:stepstick
- Q1, Q2, Q3, Q4: footprint Package_TO_SOT_SMD:SOT-23 -> Package_TO_SOT_SMD:SOT-223-3_TabPin2
Connections:
- net at Q2.1 (G): now also R3.2, R4.1
- net at Q2.2 (D): now also D3.2 (A), J_mf2.2 (Pin_2)
- net GND: now reaches Q2.3 (S)
- net GND: now also J6.15 (gnd), Q1.3 (S), Q3.3 (S), Q4.3, U1.18 (GND), U1.23 (GND), U1.28 (GND), U1.3 (GND), U1.38 (GND), C45.1, C46.2, DCDC1.2 (in+), DCDC1.4 (out+), J1.2, J14.1 (Pin_1), J2.2, J20.1 (Pin_1), J23.1 (Pin_1), J23.2 (Pin_2), J23.3 (Pin_3), J28.1 (Pin_1), J28.2 (Pin_2), J28.3 (Pin_3), J29.15 (gnd), J5.1 (Pin_1), J9.S, Q5.3 (S), R1.2, R10.2, R12.2, R4.2, R5.2, R6.2, R8.2
- net at Q4.1 (G): now also R10.1, R9.2
- net at Q4.2: now also D5.2 (A), J_mf4.2 (Pin_2)
- net stp1_en: now reaches U1.1 (GPIO0)
- net stp1_en: now also J6.1 (en)
- net endstp2: now reaches U1.10 (GPIO7)
- net endstp2: now also J14.2 (Pin_2), R6.1
- net srv1: now reaches U1.11 (GPIO8)
- net srv1: now also J10.3 (Pin_3)
- net srv2: now reaches U1.12 (GPIO9)
- net srv2: now also J3.3 (Pin_3)
- net srv3: now reaches U1.14 (GPIO10)
- net srv3: now also J4.3 (Pin_3)
- net srv4: now reaches U1.15 (GPIO11)
- net srv4: now also J11.3 (Pin_3)
- net srv5: now reaches U1.16 (GPIO12)
- net srv5: now also J15.3 (Pin_3)
- net srv6: now reaches U1.17 (GPIO13)
- net srv6: now also J16.3 (Pin_3)
- net srv7: now reaches U1.19 (GPIO14)
- net srv7: now also J17.3 (Pin_3)
- net stp1_stp: now reaches U1.2 (GPIO1)
- net stp1_stp: now also J6.7 (step)
- net srv8: now reaches U1.20 (GPIO15)
- net srv8: now also J18.3 (Pin_3)
- net MIDI_OUT: now reaches U1.21 (GPIO16)
- net MIDI_OUT: now also R23.1
- net MIDI_IN: now reaches U1.22 (GPIO17)
- net MIDI_IN: now also IC8.5, R21.1
- net mos5_gate: now reaches U1.24 (GPIO18)
- net mos5_gate: now also R11.1
- net mos4_gate: now reaches U1.25 (GPIO19)
- net mos4_gate: now also R9.1
- net mos3_gate: now reaches U1.26 (GPIO20)
- net mos3_gate: now also R7.1
- net mos2_gate: now reaches U1.27 (GPIO21)
- net mos2_gate: now also R3.1
- net mos1_gate: now reaches U1.29 (GPIO22)
- net mos1_gate: now also R2.1
- net ana2: now reaches U1.31 (GPIO26_ADC0)
- net ana2: now also J13.3 (Pin_3)
- net ana1: now reaches U1.32 (GPIO27_ADC1)
- net ana1: now also J19.3 (Pin_3)
- net GNDA: now reaches U1.33 (AGND)
- net GNDA: now also J13.1 (Pin_1), J19.1 (Pin_1)
- net ana_Vref: now reaches U1.35 (ADC_VREF)
- net ana_Vref: now also J13.2 (Pin_2), J19.2 (Pin_2)
- net +3.3V: now reaches U1.36 (3V3)
- net +3.3V: now also J6.10 (vio), J24.1 (Pin_1), J24.2 (Pin_2), J24.3 (Pin_3), J25.1 (Pin_1), J25.2 (Pin_2), J25.3 (Pin_3), J29.10 (vio)
- net +5V: now reaches U1.39 (VSYS)
- net +5V: now also D4.1 (K), D5.1 (K), D6.1 (K), DCDC1.3 (out-), J10.2 (Pin_2), J11.2 (Pin_2), J15.2 (Pin_2), J16.2 (Pin_2), J17.2 (Pin_2), J18.2 (Pin_2), J20.2 (Pin_2), J3.2 (Pin_2), J4.2 (Pin_2), J_mf3.1 (Pin_1), J_mf4.1 (Pin_1)
- net stp1_dir: now reaches U1.4 (GPIO2)
- net stp1_dir: now also J6.8 (dir)
- net stp2_en: now reaches U1.5 (GPIO3)
- net stp2_en: now also J29.1 (en)
- net stp2_stp: now reaches U1.6 (GPIO4)
- net stp2_stp: now also J29.7 (step)
- net stp2_dir: now reaches U1.7 (GPIO5)
- net stp2_dir: now also J29.8 (dir)
- net endstp1: now reaches U1.9 (GPIO6)
- net endstp1: now also J5.2 (Pin_2), R5.1
- net at J6.11 (m1b): now also J7.4 (Pin_4)
- net at J6.12 (m1a): now also J7.3 (Pin_3)
- net at J6.13 (m2a): now also J7.2 (Pin_2)
- net at J6.14 (m2b): now also J7.1 (Pin_1)
- net +24V: now reaches J6.16 (vm)
- net +24V: now also D2.1 (K), D3.1 (K), DCDC1.1 (in-), J1.1, J2.1, J29.16 (vm), J_mf1.1 (Pin_1), J_mf2.1 (Pin_1)
- net at J6.2 (ms1): now also J22.3 (Pin_3)
- net at J6.3 (ms2): now also J22.2 (Pin_2)
- net at J6.4 (sprd): now also J22.1 (Pin_1)
- net at Q3.1 (G): now also R7.2, R8.1
- net at Q3.2 (D): now also D4.2 (A), J_mf3.2 (Pin_2)
- net at Q1.1 (G): now also R1.1, R2.2
- net at Q1.2 (D): now also D2.2 (A), J_mf1.2 (Pin_2)
- new net: Q5.1 (G), R11.2, R12.1
- new net: J29.14 (m2b), J31.1 (Pin_1)
- new net: J29.13 (m2a), J31.2 (Pin_2)
- new net: J29.12 (m1a), J31.3 (Pin_3)
- new net: J29.11 (m1b), J31.4 (Pin_4)
- new net: J9.R, R20.1
- new net: C46.1, J21.S
- new net: J21.R, R22.1
- new net: D1.2 (A), IC8.2, J21.T
- new net: D1.1 (K), IC8.1, R22.2
- new net: J9.T, R23.2
- new net: J12.1 (Pin_1), J29.4 (sprd)
- new net: J12.2 (Pin_2), J29.3 (ms2)
- new net: J12.3 (Pin_3), J29.2 (ms1)
- new net +3V3: C45.2, IC8.6, R20.2, R21.2
- new net -Servo: D6.2 (A), J10.1 (Pin_1), J11.1 (Pin_1), J15.1 (Pin_1), J16.1 (Pin_1), J17.1 (Pin_1), J18.1 (Pin_1), J3.1 (Pin_1), J4.1 (Pin_1), Q5.2 (D)
Other:
- note added: "Midi"
- note added: "Mosfet1"
- note added: "Mosfet2"
- note added: "Mosfet3"
- note added: "Mosfet4"
- note added: "Mosfet_Srv"
- note added: "Pico"
- note added: "Power"
- moved on the sheet: J6, Q1, U1
